File: pcb/j0xx.kicad_pcb (KiCad board)
At the start: 2 copper layers, 73 parts, among them J1 USB_C_Receptacle, SW0 reset, SW1 SW_Push, SW10 SW_Push, SW11 SW_Push, SW12 SW_Push, SW13 SW_Push, SW14 SW_Push, SW15 SW_Push, SW16 SW_Push, SW17 SW_Push, SW18 SW_Push, SW19 SW_Push, SW2 SW_Push, SW20 SW_Push, SW3 SW_Push, SW4 SW_Push, SW5 SW_Push, SW6 SW_Push, SW7 SW_Push, SW8 SW_Push, SW9 SW_Push, U1 ATmega32U4-AU, Y1 Resonator

Commit message: First PCB draft complete
Parts:
- added C23: 0.1u, Capacitor_SMD:C_0805_2012Metric, F.Cu at (217.4, 94.6)
- added C24: 0.1u, Capacitor_SMD:C_0805_2012Metric, F.Cu at (211.7, 91.6)
- added C25: 0.1u, Capacitor_SMD:C_0805_2012Metric, F.Cu at (219.9, 108.8)
- added C26: 0.1u, Capacitor_SMD:C_0805_2012Metric, F.Cu at (199.6, 103.0)
- added C27: 0.1u, Capacitor_SMD:C_0805_2012Metric, F.Cu at (206.8, 112.5)
- added C28: 0.1u, Capacitor_SMD:C_0805_2012Metric, F.Cu at (219.9, 100.3)
- added Q1: BSS138, Package_TO_SOT_SMD:SOT-23, F.Cu at (203.4, 69.9)
- added R7: 10k, Resistor_SMD:R_0805_2012Metric, F.Cu at (205.1, 73.4)
- added R8: 10k, Resistor_SMD:R_0805_2012Metric, F.Cu at (202.3, 73.4)
- moved C21 6.55 mm to (215.9, 82.6), turned to 0 degrees
- moved R2 2.54 mm to (212.9, 78.5)
- moved R5 2.06 mm to (208.8, 78.5)
- moved R4 1.94 mm to (206.8, 78.5)
- moved F1 1.91 mm to (215.0, 78.4)
- moved Y1 0.75 mm to (202.1, 104.0)
- moved SW0 0.33 mm to (200.2, 96.8)
- moved R3 0.27 mm to (217.2, 78.5)
Connections:
- net GCCDATA renamed GCCD3.3v
- D1 pad 4: LED_DATA -> (no net)
- D20 pad 2: Net-(D20-Pad2) -> (no net)
- J1 pad A10: Net-(J1-PadA10) -> (no net)
- J1 pad A3: Net-(J1-PadA3) -> (no net)
- J1 pad A8: Net-(J1-PadA8) -> (no net)
- J1 pad B10: Net-(J1-PadB10) -> (no net)
- J1 pad B3: Net-(J1-PadB3) -> (no net)
- J1 pad B8: Net-(J1-PadB8) -> (no net)
- U1 pad 1: Net-(U1-Pad1) -> BTN_R
- U1 pad 18: BTN_START -> BTN_MODX
- U1 pad 19: BTN_R -> BTN_MODY
- U1 pad 20: BTN_Y -> BTN_START
- U1 pad 21: BTN_LS -> (no net)
- U1 pad 22: BTN_MS -> (no net)
- U1 pad 25: BTN_B -> (no net)
- U1 pad 26: BTN_X -> (no net)
- U1 pad 27: BTN_Z -> BTN_CL
- U1 pad 28: BTN_UP -> BTN_CU
- U1 pad 29: BTN_MODX -> BTN_CD
- U1 pad 30: BTN_MODY -> BTN_A
- U1 pad 31: Net-(U1-Pad31) -> BTN_CR
- U1 pad 32: Net-(U1-Pad32) -> BTN_B
- U1 pad 36: BTN_CL -> BTN_X
- U1 pad 37: BTN_CU -> BTN_Z
- U1 pad 38: BTN_CD -> BTN_UP
- U1 pad 39: BTN_A -> BTN_MS
- U1 pad 40: BTN_CR -> BTN_LS
- U1 pad 41: Net-(U1-Pad41) -> BTN_Y
- U1 pad 42: Net-(U1-Pad42) -> (no net)
- U1 pad 8: LED_DATA -> GCCD5v
Routing:
- net +5V: track 40.3 -> 1041.7 mm, vias 0 -> 10
- net LED_MODX: track 0.00 -> 257.8 mm, vias 0 -> 2
- net BTN_CD: track 0.00 -> 170.0 mm, vias 0 -> 2
- net BTN_MS: track 0.00 -> 166.3 mm
- net BTN_UP: track 0.00 -> 165.4 mm
- net BTN_L: track 0.00 -> 163.0 mm
- net BTN_A: track 0.00 -> 137.9 mm, vias 0 -> 2
- net BTN_LS: track 0.00 -> 132.3 mm
- net BTN_Z: track 0.00 -> 128.3 mm
- net BTN_LEFT: track 0.00 -> 122.4 mm
- net BTN_CR: track 0.00 -> 119.1 mm, vias 0 -> 2
- net BTN_MODX: track 0.00 -> 111.6 mm, vias 0 -> 2
- net BTN_MODY: track 0.00 -> 108.7 mm, vias 0 -> 2
- net BTN_Y: track 0.00 -> 104.5 mm
- net LED_B: track 0.00 -> 103.6 mm, vias 0 -> 2
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- added copper zone on B.Cu, net GND
- added copper zone on F.Cu, net GND
Other:
- board outline added: 316.3 x 153.1 mm

Commit message: Add dual hotswap footprint
Parts:
- SW1, SW10, SW11, SW12, SW13, SW14, SW15, SW16, SW17, SW18, SW19, SW2, SW20, SW3, SW4, SW5, SW6, SW7, SW8, SW9: footprint Button_Switch_Keyboard:SW_Cherry_MX_1.00u_PCB -> mx+choc_socket:MX+Choc_socket
- moved SW1 5.66 mm to (63.4, 119.5)
Routing:
- net BTN_L: track 163.0 -> 174.5 mm, vias 0 -> 1
- net BTN_CU: vias 2 -> 0
- net BTN_CL: vias 2 -> 0
- net BTN_CD: vias 2 -> 0
- net BTN_A: vias 2 -> 0
- net BTN_CR: vias 2 -> 0
