File: pcb/left_fingers/left_fingers.kicad_pcb (KiCad board)
At the start: 2 copper layers, 114.3 x 40.6 mm, 13 parts, among them J1 Conn_01x08, SW1 SW_Push, SW2 SW_Push, SW3 SW_Push, SW4 SW_Push

Commit message: First full iteration of physical design
Other:
- net class Default removed
