File: pcb/left_thumb/left_thumb.kicad_pcb (KiCad board)
At the start: 2 copper layers, 45.7 x 45.7 mm, 8 parts, among them J1 Conn_01x06, SW1 SW_Push, SW2 SW_Push

Commit message: First full iteration of physical design
Other:
- net class Default removed
