File: pcb/right_thumb/right_thumb.kicad_pcb (KiCad board)
At the start: 2 copper layers, 68.6 x 76.2 mm, 16 parts, among them J1 Conn_01x09, SW1 SW_Push, SW2 SW_Push, SW3 SW_Push, SW4 SW_Push, SW5 SW_Push

Commit message: First full iteration of physical design
Other:
- net class Default removed
